Commit message: 0130

File: dynamics/src/dynamics/urdf/single_arm_v12.urdf (robot description, URDF)
Before this commit: robot single_arm_v12, 8 links, 7 joints
Links:
- link Link2: mass 0.481911404914663 -> 0.46989068296361103
- link Link3: mass 0.4423890560967377 -> 0.43520591746298043
Joints:
- joint Joint3: origin xyz=0.384 0 -0.0325 rpy=0 0 0 -> xyz=0.3366413364950756 0 -0.0325 rpy=0 0 0
- joint Joint4: origin xyz=0.384 0 0.0325 rpy=0 0 3.1416 -> xyz=0.35570021785748784 0 0.0325 rpy=0 0 3.1416

File: dynamics/src/dynamics/urdf/single_arm_v12_motion.urdf (robot description, URDF)
Before this commit: robot single_arm_v12, 8 links, 7 joints
Links:
- link Link2: mass 0.481911404914663 -> 0.46989068296361103
- link Link3: mass 0.4423890560967377 -> 0.43520591746298043
Joints:
- joint Joint3: origin xyz=0.384 0 -0.0325 rpy=0 0 0 -> xyz=0.3366413364950756 0 -0.0325 rpy=0 0 0
- joint Joint4: origin xyz=0.384 0 0.0325 rpy=0 0 3.1416 -> xyz=0.35570021785748784 0 0.0325 rpy=0 0 3.1416

Commit message: 03042146

File: dynamics/src/dynamics/urdf/single_arm_v12.urdf (robot description, URDF)
Before this commit: robot single_arm_v12, 8 links, 7 joints
Links:
- link Link2: mass 0.46989068296361103 -> 0.4371547484543906
- link Link3: mass 0.43520591746298043 -> 0.44474727464934405
Joints:
- joint Joint3: origin xyz=0.3366413364950756 0 -0.0325 rpy=0 0 0 -> xyz=0.20766987261342956 0 -0.0325 rpy=0 0 0
- joint Joint4: origin xyz=0.35570021785748784 0 0.0325 rpy=0 0 3.1416 -> xyz=0.39329079538706946 0 0.0325 rpy=0 0 3.1416

File: dynamics/src/dynamics/urdf/single_arm_v12_motion.urdf (robot description, URDF)
Before this commit: robot single_arm_v12, 8 links, 7 joints
Links:
- link Link2: mass 0.46989068296361103 -> 0.4371547484543906
- link Link3: mass 0.43520591746298043 -> 0.44474727464934405
Joints:
- joint Joint3: origin xyz=0.3366413364950756 0 -0.0325 rpy=0 0 0 -> xyz=0.20766987261342956 0 -0.0325 rpy=0 0 0
- joint Joint4: origin xyz=0.35570021785748784 0 0.0325 rpy=0 0 3.1416 -> xyz=0.39329079538706946 0 0.0325 rpy=0 0 3.1416
